File: reed-sensor/reed-sensor.kicad_pcb (KiCad board)
At the start: 2 copper layers, 90 x 16 mm, 6 parts, among them J1 Conn_01x06, SW1 SW_Reed, SW2 SW_Reed

Commit message: Add gerbers, order routing
Parts:
- J1: footprint Connectors_IDC:IDC-Header_2x03_Pitch2.54mm_Straight -> Connectors_IDC:IDC-Header_2x03_Pitch2.54mm_Angled
- moved MK1 13.0 mm to (64.5, 80.0)
- moved SW2 13.0 mm to (80.0, 80.0)
- moved SW1 4.00 mm to (130.0, 80.0)
- moved MK2 3.00 mm to (106.0, 80.0)
- moved MK3 2.00 mm to (145.0, 80.0)
Routing:
- net Net-(J1-Pad5): track 0.00 -> 88.2 mm, vias 0 -> 2
- net Net-(J1-Pad3): track 0.00 -> 38.6 mm, vias 0 -> 2
- net GND: track 0.00 -> 12.8 mm, vias 0 -> 1
- added copper zone on B.Cu, net GND
- added copper zone on F.Cu, net GND
Other:
- board size 90 x 16 mm -> 111 x 16 mm
